Commit message: fixed launch file

File: adaptive_guide_description/models/adaptive_guide/adaptive_guide.urdf.xacro (robot description, xacro)
@@ -1,2 +1,3 @@
+<?xml version="1.0" ?>
 <robot name="adaptive_guide">
     <link name="world" />
@@ -70,5 +71,5 @@
         <visual>
             <geometry>
-                <mesh filename="model:///adaptive_guide/meshes/Link2.dae" />
+                <mesh filename="model://adaptive_guide/meshes/Link2.dae" />
             </geometry>
         </visual>
@@ -134,3 +135,49 @@
         <child link="EE" />
     </joint>
+    <ros2_control name="GazeboSystem" type="system">
+        <hardware>
+            <plugin>gazebo_ros2_control/GazeboSystem</plugin>
+        </hardware>
+        <joint name="joint1">
+            <command_interface name="position">
+                <param name="min">0</param>
+                <param name="max">0.1</param>
+            </command_interface>
+            <state_interface name="position"/>
+            <state_interface name="velocity"/>
+            <state_interface name="effort"/>
+        </joint>
+        <joint name="joint2">
+            <command_interface name="position">
+                <param name="min">0</param>
+                <param name="max">0.1</param>
+            </command_interface>
+            <state_interface name="position"/>
+            <state_interface name="velocity"/>
+            <state_interface name="effort"/>
+        </joint>
+        <joint name="joint3">
+            <command_interface name="position">
+                <param name="min">-0.16</param>
+                <param name="max">0</param>
+            </command_interface>
+            <state_interface name="position"/>
+            <state_interface name="velocity"/>
+            <state_interface name="effort"/>
+        </joint>
+        <joint name="joint4">
+            <command_interface name="position">
+                <param name="min">-3</param>
+                <param name="max">3</param>
+            </command_interface>
+            <state_interface name="position"/>
+            <state_interface name="velocity"/>
+            <state_interface name="effort"/>
+        </joint>
+    </ros2_control>
+    <gazebo>
+        <plugin filename="libgazebo_ros2_control.so" name="gazebo_ros2_control">
+            <parameters>$(find needle_path_control)/config/needle_controller.yaml</parameters>
+        </plugin>
+    </gazebo>
 </robot>

Commit message: changed initial needle depth position

File: adaptive_guide_description/models/adaptive_guide/adaptive_guide.urdf.xacro (robot description, xacro)
@@ -129,6 +129,6 @@
     </joint>
     <joint name="joint3" type="prismatic">
-        <origin xyz="0.045724 0.009758 0.0333375" rpy="0 0 0 " />
-        <limit lower="-0.160" upper="0" effort="30.0" velocity="6" />
+        <origin xyz="0.045724 -0.169758 0.0333375" rpy="0 0 0 " />
+        <limit lower="-0.0" upper="0.16" effort="30.0" velocity="6" />
         <parent link="link2" />
         <child link="link3" />
@@ -171,6 +171,6 @@
         <joint name="joint3">
             <command_interface name="position">
-                <param name="min">-0.16</param>
-                <param name="max">0</param>
+                <param name="min">0</param>
+                <param name="max">0.16</param>
             </command_interface>
             <state_interface name="position"/>
